Commit message: tripod gait

File: install/hexapod_description/share/hexapod_description/urdf/hexapod.urdf (robot description, URDF)
Before this commit: robot hexapod, 27 links, 26 joints
Joints:
- joint ankle_2_joint: limit lower=-1.5708 upper=1.5708 effort=10.0 velocity=0.1 -> lower=-1.5708 upper=1.5708 effort=5.0 velocity=5.0
- joint ankle_3_joint: limit lower=-1.5708 upper=1.5708 effort=10.0 velocity=0.1 -> lower=-1.5708 upper=1.5708 effort=5.0 velocity=5.0
- joint ankle_4_joint: limit lower=-1.5708 upper=1.5708 effort=10.0 velocity=0.1 -> lower=-1.5708 upper=1.5708 effort=5.0 velocity=5.0
- joint ankle_5_joint: limit lower=-1.5708 upper=1.5708 effort=10.0 velocity=0.1 -> lower=-1.5708 upper=1.5708 effort=5.0 velocity=5.0
- joint ankle_6_joint: limit lower=-1.5708 upper=1.5708 effort=10.0 velocity=0.1 -> lower=-1.5708 upper=1.5708 effort=5.0 velocity=5.0
- joint hip_1_joint: axis 0 0 -1 -> 0 0 1; limit lower=-1.5708 upper=1.5708 effort=10.0 velocity=0.1 -> lower=1.5708 upper=-1.5708 effort=5.0 velocity=5.0
- joint hip_2_joint: limit lower=-1.5708 upper=1.5708 effort=10.0 velocity=0.1 -> lower=-1.5708 upper=1.5708 effort=5.0 velocity=5.0
- joint hip_3_joint: axis 0 0 -1 -> 0 0 1; limit lower=-1.5708 upper=1.5708 effort=10.0 velocity=0.1 -> lower=1.5708 upper=-1.5708 effort=5.0 velocity=5.0
- joint hip_4_joint: limit lower=-1.5708 upper=1.5708 effort=10.0 velocity=0.1 -> lower=-1.5708 upper=1.5708 effort=5.0 velocity=5.0
- joint hip_5_joint: limit lower=-1.5708 upper=1.5708 effort=10.0 velocity=0.1 -> lower=-1.5708 upper=1.5708 effort=5.0 velocity=5.0
- joint hip_6_joint: limit lower=-1.5708 upper=1.5708 effort=10.0 velocity=0.1 -> lower=-1.5708 upper=1.5708 effort=5.0 velocity=5.0
- joint knee_1_joint: limit lower=-1.5708 upper=1.5708 effort=10.0 velocity=0.1 -> lower=-1.5708 upper=1.5708 effort=5.0 velocity=5.0
- joint knee_2_joint: limit lower=-1.5708 upper=1.5708 effort=10.0 velocity=0.1 -> lower=-1.5708 upper=1.5708 effort=5.0 velocity=5.0
- joint knee_3_joint: limit lower=-1.5708 upper=1.5708 effort=10.0 velocity=0.1 -> lower=-1.5708 upper=1.5708 effort=5.0 velocity=5.0
- joint knee_4_joint: limit lower=-1.5708 upper=1.5708 effort=10.0 velocity=0.1 -> lower=-1.5708 upper=1.5708 effort=5.0 velocity=5.0
- joint knee_5_joint: limit lower=-1.5708 upper=1.5708 effort=10.0 velocity=0.1 -> lower=-1.5708 upper=1.5708 effort=5.0 velocity=5.0
- joint knee_6_joint: limit lower=-1.5708 upper=1.5708 effort=10.0 velocity=0.1 -> lower=-1.5708 upper=1.5708 effort=5.0 velocity=5.0

Commit message: simulation

File: install/hexapod_description/share/hexapod_description/urdf/hexapod.urdf (robot description, URDF)
Before this commit: robot hexapod, 27 links, 26 joints
Links:
- removed link T260_link
- removed link realsense_link
- removed link tip_1_link
- removed link tip_2_link
- removed link tip_3_link
- removed link tip_4_link
- removed link tip_5_link
- removed link tip_6_link
- link ankle_1_link: mass 0.062766 -> 0.058138; geometry collision mesh filename=package://my_robot/meshes/ankle_1_link.STL; visual mesh filename=package://my_robot/meshes/ankle_1_link.STL
- link ankle_2_link: mass 0.062766 -> 0.058138; geometry collision mesh filename=package://my_robot/meshes/ankle_2_link.STL; visual mesh filename=package://my_robot/meshes/ankle_2_link.STL
- link ankle_3_link: mass 0.0627656309071367 -> 0.058138; geometry collision mesh filename=package://my_robot/meshes/ankle_3_link.STL; visual mesh filename=package://my_robot/meshes/ankle_3_link.STL
- link ankle_4_link: mass 0.0627656309071365 -> 0.0581378722016232; geometry collision mesh filename=package://my_robot/meshes/ankle_4_link.STL; visual mesh filename=package://my_robot/meshes/ankle_4_link.STL
- link ankle_5_link: mass 0.0627655365921658 -> 0.058138; geometry collision mesh filename=package://my_robot/meshes/ankle_5_link.STL; visual mesh filename=package://my_robot/meshes/ankle_5_link.STL
- link ankle_6_link: mass 0.0627656309071363 -> 0.058138; geometry collision mesh filename=package://my_robot/meshes/ankle_6_link.STL; visual mesh filename=package://my_robot/meshes/ankle_6_link.STL
- link base_link: mass 0.41864 -> 0.16098; geometry collision mesh filename=package://my_robot/meshes/base_link.STL; visual mesh filename=package://my_robot/meshes/base_link.STL
- link hip_1_link: mass 0.028857 -> 0.0982; geometry collision mesh filename=package://my_robot/meshes/hip_1_link.STL; visual mesh filename=package://my_robot/meshes/hip_1_link.STL
- link hip_2_link: mass 0.0288571734423381 -> 0.0982; geometry collision mesh filename=package://my_robot/meshes/hip_2_link.STL; visual mesh filename=package://my_robot/meshes/hip_2_link.STL
- link hip_3_link: mass 0.028857126372038 -> 0.0982; geometry collision mesh filename=package://my_robot/meshes/hip_3_link.STL; visual mesh filename=package://my_robot/meshes/hip_3_link.STL
- link hip_4_link: mass 0.028857126372038 -> 0.0982; geometry collision mesh filename=package://my_robot/meshes/hip_4_link.STL; visual mesh filename=package://my_robot/meshes/hip_4_link.STL
- link hip_5_link: mass 0.0288571734423381 -> 0.0982; geometry collision mesh filename=package://my_robot/meshes/hip_5_link.STL; visual mesh filename=package://my_robot/meshes/hip_5_link.STL
- link hip_6_link: mass 0.028857126372038 -> 0.0982; geometry collision mesh filename=package://my_robot/meshes/hip_6_link.STL; visual mesh filename=package://my_robot/meshes/hip_6_link.STL
- link knee_1_link: mass 0.058628 -> 0.0019497; geometry collision mesh filename=package://my_robot/meshes/knee_1_link.STL; visual mesh filename=package://my_robot/meshes/knee_1_link.STL
- link knee_2_link: mass 0.058628 -> 0.0019022; geometry collision mesh filename=package://my_robot/meshes/knee_2_link.STL; visual mesh filename=package://my_robot/meshes/knee_2_link.STL
- link knee_3_link: mass 0.0586281827753225 -> 0.0019022; geometry collision mesh filename=package://my_robot/meshes/knee_3_link.STL; visual mesh filename=package://my_robot/meshes/knee_3_link.STL
- link knee_4_link: mass 0.0586281825189454 -> 0.0019022; geometry collision mesh filename=package://my_robot/meshes/knee_4_link.STL; visual mesh filename=package://my_robot/meshes/knee_4_link.STL
- link knee_5_link: mass 0.0586281862879415 -> 0.0019022; geometry collision mesh filename=package://my_robot/meshes/knee_5_link.STL; visual mesh filename=package://my_robot/meshes/knee_5_link.STL
- link knee_6_link: mass 0.0586281825189454 -> 0.0982; geometry collision mesh filename=package://my_robot/meshes/knee_6_link.STL; visual mesh filename=package://my_robot/meshes/knee_6_link.STL
Joints:
- removed joint T260_joint
- removed joint realsense_joint
- removed joint tip_1_joint
- removed joint tip_2_joint
- removed joint tip_3_joint
- removed joint tip_4_joint
- removed joint tip_5_joint
- removed joint tip_6_joint
- joint ankle_1_joint: axis 0 0 -1 -> 0 0 1; limit lower=-1.5708 upper=1.5708 effort=10.0 velocity=0.1 -> (none); origin xyz=-0.065 -0.015 6E-05 rpy=0 0 1.1778 -> xyz=0 0 0.0209 rpy=0 0 0; type revolute -> fixed
- joint ankle_2_joint: axis 0 0 -1 -> 0 0 1; limit lower=-1.5708 upper=1.5708 effort=5.0 velocity=5.0 -> (none); origin xyz=-0.065 -0.015 6E-05 rpy=0 0 1.1778 -> xyz=0 0 0.0209 rpy=0 0 0; type revolute -> fixed
- joint ankle_3_joint: axis 0 0 -1 -> 0 0 0; limit lower=-1.5708 upper=1.5708 effort=5.0 velocity=5.0 -> (none); origin xyz=-0.065 -0.015 6E-05 rpy=0 0 1.1778 -> xyz=0 0 0.0209 rpy=0 0 0; type revolute -> fixed
- joint ankle_4_joint: limit lower=-1.5708 upper=1.5708 effort=5.0 velocity=5.0 -> (none); origin xyz=0.065 -0.015 -6E-05 rpy=0 0 -1.1778 -> xyz=0 0 0.0209 rpy=0 0 0; type revolute -> fixed
- joint ankle_5_joint: axis 0 0 1 -> 0 0 0; limit lower=-1.5708 upper=1.5708 effort=5.0 velocity=5.0 -> (none); origin xyz=0.065 -0.015 -6E-05 rpy=0 0 -1.1778 -> xyz=0 0 0.020899999963091 rpy=0 0 0; type revolute -> fixed
- joint ankle_6_joint: limit lower=-1.5708 upper=1.5708 effort=5.0 velocity=5.0 -> (none); origin xyz=0.065 -0.015 -6E-05 rpy=0 0 -1.1778 -> xyz=0 0 0.0208999999630915 rpy=0 0 0; type revolute -> fixed
- joint hip_1_joint: axis 0 0 1 -> 0 0 -1; limit lower=1.5708 upper=-1.5708 effort=5.0 velocity=5.0 -> lower=-1.5708 upper=1.5708 effort=10 velocity=1; origin xyz=0.11551 -0.065506 0.01594 rpy=0 0 0.74171 -> xyz=0.0777 -0.034784 0.022207 rpy=-0.0098734 -0.0098729 -0.78535
- joint hip_2_joint: axis -0.015899 0.015899 0.99975 -> 0 0 -1; limit lower=-1.5708 upper=1.5708 effort=5.0 velocity=5.0 -> lower=-1.5708 upper=1.5708 effort=10 velocity=1; origin xyz=0 -0.06978 0.01594 rpy=0 0 -0.043686 -> xyz=-0.0032327 -0.075288 0.018972 rpy=-0.003614 -0.013487 -1.309
- joint hip_3_joint: axis 0 0 1 -> 0 0 -1; limit lower=1.5708 upper=-1.5708 effort=5.0 velocity=5.0 -> lower=-1.5708 upper=1.5708 effort=10 velocity=1; origin xyz=-0.11551 -0.065506 0.01594 rpy=0 0 -0.82908 -> xyz=-0.0737 -0.034784 0.022207 rpy=0.0098734 -0.0098729 -2.3562
- joint hip_4_joint: axis 0 0 -1 -> 0 0 1; limit lower=-1.5708 upper=1.5708 effort=5.0 velocity=5.0 -> lower=-1.5708 upper=1.5708 effort=10 velocity=1; origin xyz=0.11551 0.065506 0.01594 rpy=0 0 -0.82908 -> xyz=0.0777 0.03521 0.021229 rpy=-0.0098734 0.0098729 0.78535
- joint hip_5_joint: limit lower=-1.5708 upper=1.5708 effort=5.0 velocity=5.0 -> lower=1.5708 upper=-1.5708 effort=10 velocity=1; origin xyz=0 0.06978 0.01594 rpy=0 0 -0.043686 -> xyz=-0.0032327 0.075608 0.016865 rpy=-0.003614 0.013487 1.309
- joint hip_6_joint: limit lower=-1.5708 upper=1.5708 effort=5.0 velocity=5.0 -> lower=1.5708 upper=-1.5708 effort=10 velocity=1; origin xyz=-0.11551 0.065506 0.01594 rpy=0 0 0.74171 -> xyz=-0.0737 0.03521 0.021229 rpy=0.0098734 0.0098729 2.3562
- joint knee_1_joint: limit lower=-1.5708 upper=1.5708 effort=5.0 velocity=5.0 -> lower=-1.5708 upper=1.5708 effort=10 velocity=1; origin xyz=0 -0.052 0 rpy=1.5708 0.64175 1.5708 -> xyz=0.024 0.0209 -0.0209 rpy=1.5708 0 0
- joint knee_2_joint: limit lower=-1.5708 upper=1.5708 effort=5.0 velocity=5.0 -> lower=-1.5708 upper=1.5708 effort=10 velocity=1; origin xyz=0 -0.052 0 rpy=1.5708 0.64175 1.5708 -> xyz=0.024 0.0209 -0.0209 rpy=1.5708 0 0
- joint knee_3_joint: limit lower=-1.5708 upper=1.5708 effort=5.0 velocity=5.0 -> lower=-1.5708 upper=1.5708 effort=10 velocity=1; origin xyz=0 -0.052 0 rpy=1.5708 0.64175 1.5708 -> xyz=0.024 0.0209 -0.0209 rpy=1.5708 0 0
- joint knee_4_joint: axis 0 0 -1 -> 0 0 1; limit lower=-1.5708 upper=1.5708 effort=5.0 velocity=5.0 -> lower=-1.5708 upper=1.5708 effort=10 velocity=1; origin xyz=0 0.052 0 rpy=1.5708 -0.64175 1.5708 -> xyz=0.024 0.0209 -0.0209 rpy=1.5708 0 0
- joint knee_5_joint: axis 0 0 -1 -> 0 0 1; limit lower=-1.5708 upper=1.5708 effort=5.0 velocity=5.0 -> lower=-1.5708 upper=1.5708 effort=10 velocity=1; origin xyz=0 0.052 0 rpy=1.5708 -0.64175 1.5708 -> xyz=0.024 0.0209 -0.0209 rpy=1.5708 0 0
- joint knee_6_joint: axis 0 0 -1 -> 0 0 1; limit lower=-1.5708 upper=1.5708 effort=5.0 velocity=5.0 -> lower=-1.5708 upper=1.5708 effort=10 velocity=1; origin xyz=0 0.052 0 rpy=1.5708 -0.64175 1.5708 -> xyz=0.024 0.0209 -0.0209 rpy=1.5708 0 0
